Commit message: moveit errors

File: src/my_arm_description/urdf/my_arm_puma.urdf.xacro (robot description, xacro)
@@ -214,4 +214,30 @@
   </joint>
   <!-- =========================
+       Tool / TCP frame
+       ========================= -->
+  <xacro:arg name="tool_z" default="0.15"/>
+  <xacro:property name="tool_z" value="$(arg tool_z)"/>
+  <link name="puma_tool">
+    <visual>
+      <origin xyz="0 0 ${tool_z/2.0}" rpy="0 0 0"/>
+      <geometry>
+        <cylinder radius="0.015" length="${tool_z}"/>
+      </geometry>
+      <material name="dark"/>
+    </visual>
+    <collision>
+      <origin xyz="0 0 ${tool_z/2.0}" rpy="0 0 0"/>
+      <geometry>
+        <cylinder radius="0.015" length="${tool_z}"/>
+      </geometry>
+    </collision>
+    <xacro:inertial_cylinder_z mass="0.02" radius="0.015" length="${tool_z}"/>
+  </link>
+  <joint name="link6_to_puma_tool" type="fixed">
+    <parent link="link6"/>
+    <child link="puma_tool"/>
+    <origin xyz="0 0 ${tool_z}" rpy="0 0 0"/>
+  </joint>
+  <!-- =========================
        ros2_control (gz_ros2_control)
        ========================= -->

Commit message: moveit modified

File: src/my_arm_description/urdf/my_arm_puma.urdf.xacro (robot description, xacro)
@@ -214,29 +214,31 @@
   </joint>
   <!-- =========================
-       Tool / TCP frame
-       ========================= -->
-  <xacro:arg name="tool_z" default="0.15"/>
-  <xacro:property name="tool_z" value="$(arg tool_z)"/>
-  <link name="puma_tool">
-    <visual>
-      <origin xyz="0 0 ${tool_z/2.0}" rpy="0 0 0"/>
-      <geometry>
-        <cylinder radius="0.015" length="${tool_z}"/>
-      </geometry>
-      <material name="dark"/>
-    </visual>
-    <collision>
-      <origin xyz="0 0 ${tool_z/2.0}" rpy="0 0 0"/>
-      <geometry>
-        <cylinder radius="0.015" length="${tool_z}"/>
-      </geometry>
-    </collision>
-    <xacro:inertial_cylinder_z mass="0.02" radius="0.015" length="${tool_z}"/>
-  </link>
-  <joint name="link6_to_puma_tool" type="fixed">
+     Tool / TCP frame
+     ========================= -->
+    <xacro:arg name="tool_z" default="0.15"/>
+    <xacro:arg name="tool_radius" default="0.02"/>
+    <xacro:property name="tool_z" value="$(arg tool_z)"/>
+    <xacro:property name="tool_radius" value="$(arg tool_radius)"/>
+    <link name="puma_tool">
+    <visual>
+        <origin xyz="0 0 0" rpy="0 0 0"/>
+        <geometry>
+        <sphere radius="${tool_radius}"/>
+        </geometry>
+        <material name="dark"/>
+    </visual>
+    <collision>
+        <origin xyz="0 0 0" rpy="0 0 0"/>
+        <geometry>
+        <sphere radius="${tool_radius}"/>
+        </geometry>
+    </collision>
+    <xacro:inertial_sphere mass="0.001" radius="${tool_radius}"/>
+    </link>
+    <joint name="link6_to_puma_tool" type="fixed">
     <parent link="link6"/>
     <child link="puma_tool"/>
     <origin xyz="0 0 ${tool_z}" rpy="0 0 0"/>
-  </joint>
+    </joint>
   <!-- =========================
        ros2_control (gz_ros2_control)
@@ -244,5 +246,5 @@
   <ros2_control name="MyArmSystem" type="system">
     <hardware>
-      <plugin>gz_ros2_control/GazeboSimSystem</plugin>
+      <plugin>ign_ros2_control/IgnitionSystem</plugin>
     </hardware>
     <joint name="joint1">

Commit message: arm_pose

File: src/my_arm_description/urdf/my_arm_puma.urdf.xacro (robot description, xacro)
@@ -220,5 +220,5 @@
     <xacro:property name="tool_z" value="$(arg tool_z)"/>
     <xacro:property name="tool_radius" value="$(arg tool_radius)"/>
-    <link name="puma_tool">
+    <link name="tool">
     <visual>
         <origin xyz="0 0 0" rpy="0 0 0"/>
@@ -236,7 +236,7 @@
     <xacro:inertial_sphere mass="0.001" radius="${tool_radius}"/>
     </link>
-    <joint name="link6_to_puma_tool" type="fixed">
+    <joint name="link6_to_tool" type="fixed">
     <parent link="link6"/>
-    <child link="puma_tool"/>
+    <child link="tool"/>
     <origin xyz="0 0 ${tool_z}" rpy="0 0 0"/>
     </joint>

File: src/my_arm_description/urdf/my_arm_ur5e.urdf.xacro (robot description, xacro)
@@ -249,5 +249,5 @@
     <child link="link2"/>
     <origin xyz="0 0 $(arg d1)" rpy="0 0 0"/>
-    <axis xyz="0 1 0"/>
+    <axis xyz="0 -1 0"/>
     <limit lower="-6.28318530718" upper="6.28318530718" effort="$(arg joint_effort)" velocity="$(arg joint_vel)"/>
     <dynamics damping="2.0" friction="0.0"/>
@@ -258,5 +258,5 @@
     <child link="link3"/>
     <origin xyz="-$(arg a2) 0 0" rpy="0 0 0"/>
-    <axis xyz="0 1 0"/>
+    <axis xyz="0 -1 0"/>
     <limit lower="-6.28318530718" upper="6.28318530718" effort="$(arg joint_effort)" velocity="$(arg joint_vel)"/>
     <dynamics damping="2.0" friction="0.0"/>
@@ -267,5 +267,5 @@
     <child link="link4"/>
     <origin xyz="-$(arg a3) 0 0" rpy="0 0 0"/>
-    <axis xyz="0 1 0"/>
+    <axis xyz="0 -1 0"/>
     <limit lower="-6.28318530718" upper="6.28318530718" effort="$(arg joint_effort)" velocity="$(arg joint_vel)"/>
     <dynamics damping="1.0" friction="0.0"/>
@@ -276,5 +276,5 @@
     <child link="link5"/>
     <origin xyz="0 -$(arg d4) 0" rpy="0 0 0"/>
-    <axis xyz="0 0 1"/>
+    <axis xyz="0 0 -1"/>
     <limit lower="-6.28318530718" upper="6.28318530718" effort="$(arg joint_effort)" velocity="$(arg joint_vel)"/>
     <dynamics damping="1.0" friction="0.0"/>
@@ -285,10 +285,10 @@
     <child link="link6"/>
     <origin xyz="0 0 -$(arg d5)" rpy="0 0 0"/>
-    <axis xyz="0 1 0"/>
+    <axis xyz="0 -1 0"/>
     <limit lower="-6.28318530718" upper="6.28318530718" effort="$(arg joint_effort)" velocity="$(arg joint_vel)"/>
     <dynamics damping="0.8" friction="0.0"/>
   </joint>
   <!-- Tool frame: small sphere 15 cm along -Y from link6 frame -->
-  <link name="ur5e_tool">
+  <link name="tool">
     <visual>
       <origin xyz="0 0 0" rpy="0 0 0"/>
@@ -316,7 +316,7 @@
     </inertial>
   </link>
-  <joint name="link6_to_ur5e_tool" type="fixed">
+  <joint name="link6_to_tool" type="fixed">
     <parent link="link6"/>
-    <child link="ur5e_tool"/>
+    <child link="tool"/>
     <origin xyz="0 -0.15 0" rpy="0 0 0"/>
   </joint>
