Commit message: added ur5e_moveit_config

File: src/my_arm_description/urdf/my_arm_ur5e.urdf.xacro (robot description, xacro)
@@ -199,4 +199,36 @@
     <dynamics damping="0.8" friction="0.0"/>
   </joint>
+  <!-- Tool frame: small sphere 15 cm along -Y from link6 frame -->
+  <link name="ur5e_tool">
+    <visual>
+      <origin xyz="0 0 0" rpy="0 0 0"/>
+      <geometry>
+        <sphere radius="0.01"/>
+      </geometry>
+      <material name="dark"/>
+    </visual>
+    <collision>
+      <origin xyz="0 0 0" rpy="0 0 0"/>
+      <geometry>
+        <sphere radius="0.01"/>
+      </geometry>
+    </collision>
+    <inertial>
+        <mass value="0.01"/>
+        <origin xyz="0 0 0" rpy="0 0 0"/>
+        <inertia
+        ixx="0.000001"
+        ixy="0.0"
+        ixz="0.0"
+        iyy="0.000001"
+        iyz="0.0"
+        izz="0.000001"/>
+    </inertial>
+  </link>
+  <joint name="link6_to_ur5e_tool" type="fixed">
+    <parent link="link6"/>
+    <child link="ur5e_tool"/>
+    <origin xyz="0 -0.15 0" rpy="0 0 0"/>
+  </joint>
   <!--
        ros2_control (gz_ros2_control)

Commit message: added surface

File: src/my_arm_description/urdf/my_arm_ur5e.urdf.xacro (robot description, xacro)
@@ -73,4 +73,94 @@
     <origin xyz="0 0 0" rpy="0 0 0"/>
   </joint>
+    <!-- Reference floor: 1.2 m x 1.2 m centered at base_link -->
+    <link name="reference_floor">
+    <visual>
+        <origin xyz="0 0 -0.005" rpy="0 0 0"/>
+        <geometry>
+        <box size="1.2 1.2 0.01"/>
+        </geometry>
+        <material name="brown">
+        <color rgba="0.45 0.25 0.10 1.0"/>
+        </material>
+    </visual>
+    <collision>
+        <origin xyz="0 0 -0.005" rpy="0 0 0"/>
+        <geometry>
+        <box size="1.2 1.2 0.01"/>
+        </geometry>
+    </collision>
+    <inertial>
+        <mass value="0.1"/>
+        <origin xyz="0 0 -0.005" rpy="0 0 0"/>
+        <inertia ixx="0.012" ixy="0" ixz="0"
+                iyy="0.012" iyz="0"
+                izz="0.024"/>
+    </inertial>
+    </link>
+    <joint name="world_to_reference_floor" type="fixed">
+    <parent link="world"/>
+    <child link="reference_floor"/>
+    <origin xyz="0 0 0" rpy="0 0 0"/>
+    </joint>
+    <!-- X axis: red, 30 cm long, 1 cm thick -->
+    <link name="x_axis_ref">
+    <visual>
+        <origin xyz="0.15 0 0.01" rpy="0 1.57079632679 0"/>
+        <geometry>
+        <cylinder radius="0.005" length="0.30"/>
+        </geometry>
+        <material name="red">
+        <color rgba="1.0 0.0 0.0 1.0"/>
+        </material>
+    </visual>
+    <collision>
+        <origin xyz="0.15 0 0.01" rpy="0 1.57079632679 0"/>
+        <geometry>
+        <cylinder radius="0.005" length="0.30"/>
+        </geometry>
+    </collision>
+    <inertial>
+        <mass value="0.01"/>
+        <origin xyz="0.15 0 0.01" rpy="0 1.57079632679 0"/>
+        <inertia ixx="0.000001" ixy="0" ixz="0"
+                iyy="0.000001" iyz="0"
+                izz="0.000001"/>
+    </inertial>
+    </link>
+    <joint name="world_to_x_axis_ref" type="fixed">
+    <parent link="world"/>
+    <child link="x_axis_ref"/>
+    <origin xyz="0 0 0" rpy="0 0 0"/>
+    </joint>
+    <!-- Y axis: green, 30 cm long, 1 cm thick -->
+    <link name="y_axis_ref">
+    <visual>
+        <origin xyz="0 0.15 0.015" rpy="1.57079632679 0 0"/>
+        <geometry>
+        <cylinder radius="0.005" length="0.30"/>
+        </geometry>
+        <material name="green">
+        <color rgba="0.0 0.8 0.0 1.0"/>
+        </material>
+    </visual>
+    <collision>
+        <origin xyz="0 0.15 0.015" rpy="1.57079632679 0 0"/>
+        <geometry>
+        <cylinder radius="0.005" length="0.30"/>
+        </geometry>
+    </collision>
+    <inertial>
+        <mass value="0.01"/>
+        <origin xyz="0 0.15 0.015" rpy="1.57079632679 0 0"/>
+        <inertia ixx="0.000001" ixy="0" ixz="0"
+                iyy="0.000001" iyz="0"
+                izz="0.000001"/>
+    </inertial>
+    </link>
+    <joint name="world_to_y_axis_ref" type="fixed">
+    <parent link="world"/>
+    <child link="y_axis_ref"/>
+    <origin xyz="0 0 0" rpy="0 0 0"/>
+    </joint>
   <link name="base_link">
     <visual>

Commit message: sequences

File: src/my_arm_description/urdf/my_arm_ur5e.urdf.xacro (robot description, xacro)
@@ -319,5 +319,5 @@
     <parent link="link6"/>
     <child link="tool"/>
-    <origin xyz="0 -0.15 0" rpy="0 0 0"/>
+    <origin xyz="0 -0.15 0" rpy="1.5708 0 0"/>
   </joint>
   <!--
